File: rev1/acrylic/framework-acrylic-base.kicad_pcb (KiCad board)
At the start: 2 copper layers, 238.1 x 133.4 mm, 0 parts

Commit message: add acrylic cover + update schematic pdf
Other:
- outline, holes or cut-outs redrawn
Changed lines of the file:
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@@
   (general
     (thickness 1.6)
-    (drawings 119)
+    (drawings 128)
     (tracks 0)
     (zones 0)
@@
     (solder_mask_min_width 0.25)
     (aux_axis_origin 0 0)
-    (grid_origin 36.308625 154.057625)
+    (grid_origin 151.79925 56.426375)
     (visible_elements 7FFFF77F)
     (pcbplotparams
@@
     (diff_pair_gap 0.25)
   )
+  (gr_line (start 262.52784 30.232515) (end 262.52784 34.995035) (layer Edge.Cuts) (width 0.05))
+  (gr_arc (start 260.14658 30.232515) (end 262.52784 30.232515) (angle -90) (layer Edge.Cuts) (width 0.05))
+  (gr_line (start 42.26129 27.851255) (end 52.977375 27.851375) (layer Edge.Cuts) (width 0.05))
+  (gr_line (start 39.88003 49.282595) (end 39.88003 30.232515) (layer Edge.Cuts) (width 0.05))
+  (gr_arc (start 42.26129 30.232515) (end 42.26129 27.851255) (angle -90) (layer Edge.Cuts) (width 0.05))
+  (gr_line (start 260.14658 37.376295) (end 238.71524 37.376295) (layer Edge.Cuts) (width 0.05))
+  (gr_line (start 233.95272 52.854485) (end 158.94303 52.854485) (layer Edge.Cuts) (width 0.05))
+  (gr_line (start 236.33398 39.757555) (end 236.33398 50.473225) (layer Edge.Cuts) (width 0.05))
+  (gr_arc (start 233.95272 50.473225) (end 233.95272 52.854485) (angle -90) (layer Edge.Cuts) (width 0.05))
+  (gr_arc (start 238.71524 39.757555) (end 238.71524 37.376295) (angle -90) (layer Edge.Cuts) (width 0.05))
+  (gr_arc (start 260.14658 34.995035) (end 260.14658 37.376295) (angle -90) (layer Edge.Cuts) (width 0.05))
+  (gr_line (start 264.9091 51.663855) (end 254.19343 51.663855) (layer Edge.Cuts) (width 0.05))
+  (gr_line (start 267.289875 58.807625) (end 267.29036 54.045115) (layer Edge.Cuts) (width 0.05))
+  (gr_line (start 251.810485 56.426375) (end 251.81217 54.045115) (layer Edge.Cuts) (width 0.05))
+  (gr_arc (start 254.19343 54.045115) (end 254.19343 51.663855) (angle -90) (layer Edge.Cuts) (width 0.05))
+  (gr_arc (start 264.9091 54.045115) (end 267.29036 54.045115) (angle -90) (layer Edge.Cuts) (width 0.05))
+  (gr_line (start 43.45192 52.854485) (end 144.65547 52.854485) (layer Edge.Cuts) (width 0.05))
+  (gr_line (start 155.37114 49.282595) (end 155.37114 48.091965) (layer Edge.Cuts) (width 0.05))
+  (gr_line (start 148.22736 49.282595) (end 148.22736 48.091965) (layer Edge.Cuts) (width 0.05))
+  (gr_arc (start 144.65547 49.282595) (end 144.65547 52.854485) (angle -90) (layer Edge.Cuts) (width 0.05))
+  (gr_arc (start 158.94303 49.282595) (end 155.37114 49.282595) (angle -90) (layer Edge.Cuts) (width 0.05))
+  (gr_arc (start 151.79925 48.091965) (end 155.37114 48.091965) (angle -180) (layer Edge.Cuts) (width 0.05))
+  (gr_arc (start 43.45192 49.282595) (end 39.88003 49.282595) (angle -90) (layer Edge.Cuts) (width 0.05))
+  (gr_circle (center 267.29036 49.282595) (end 268.39036 49.282595) (layer Edge.Cuts) (width 0.05))
+  (gr_circle (center 151.79925 48.091965) (end 152.89925 48.091965) (layer Edge.Cuts) (width 0.05))
+  (gr_circle (center 36.30814 49.282595) (end 37.40814 49.282595) (layer Edge.Cuts) (width 0.05))
   (gr_circle (center 36.308625 154.057625) (end 37.408625 154.057625) (layer Edge.Cuts) (width 0.05))
   (gr_circle (center 36.308625 56.426375) (end 37.408625 56.426375) (layer Edge.Cuts) (width 0.05))
@@
   (gr_line (start 253.002375 71.9045) (end 263.718 71.9045) (layer Edge.Cuts) (width 0.05))
   (gr_line (start 268.4805 64.76075) (end 268.4805 59.99825) (layer Edge.Cuts) (width 0.05))
-  (gr_line (start 267.289875 58.807625) (end 267.289875 48.092) (layer Edge.Cuts) (width 0.05))
-  (gr_line (start 264.908625 45.71075) (end 254.193 45.71075) (layer Edge.Cuts) (width 0.05))
-  (gr_line (start 251.81175 48.092) (end 251.810485 56.426375) (layer Edge.Cuts) (width 0.05))
   (gr_arc (start 248.239875 56.426375) (end 245.579252 58.807623) (angle -138.1715706) (layer Edge.Cuts) (width 0.05))
   (gr_line (start 267.289875 68.332625) (end 267.289875 65.951375) (layer Edge.Cuts) (width 0.05))
@@
   (gr_arc (start 267.289875 64.76075) (end 267.289875 65.951375) (angle -90) (layer Edge.Cuts) (width 0.05))
   (gr_arc (start 267.289875 59.99825) (end 268.4805 59.99825) (angle -90) (layer Edge.Cuts) (width 0.05))
-  (gr_line (start 231.571125 27.851375) (end 263.718 27.851375) (layer Edge.Cuts) (width 0.05))
+  (gr_line (start 231.571125 27.851375) (end 260.14658 27.851375) (layer Edge.Cuts) (width 0.05))
   (gr_line (start 157.752375 27.851375) (end 177.993 27.851375) (layer Edge.Cuts) (width 0.05))
   (gr_line (start 125.6055 27.851375) (end 145.846125 27.851375) (layer Edge.Cuts) (width 0.05))
   (gr_line (start 63.693 27.851375) (end 72.027375 27.851375) (layer Edge.Cuts) (width 0.05))
-  (gr_line (start 39.8805 27.851375) (end 52.977375 27.851375) (layer Edge.Cuts) (width 0.05))
   (gr_line (start 179.183625 26.66075) (end 230.3805 26.66075) (layer Edge.Cuts) (width 0.05))
   (gr_line (start 147.03675 26.66075) (end 156.56175 26.66075) (layer Edge.Cuts) (width 0.05))
@@
   (gr_line (start 38.689875 127.863875) (end 264.908625 127.863875) (layer Edge.Cuts) (width 0.05))
   (gr_arc (start 38.689875 125.482625) (end 36.308625 125.482625) (angle -90) (layer Edge.Cuts) (width 0.05))
-  (gr_arc (start 264.908625 48.092) (end 267.289875 48.092) (angle -90) (layer Edge.Cuts) (width 0.05))
-  (gr_line (start 267.289875 37.376375) (end 267.289875 31.42325) (layer Edge.Cuts) (width 0.05))
-  (gr_arc (start 264.908625 37.376375) (end 264.908625 39.757625) (angle -90) (layer Edge.Cuts) (width 0.05))
-  (gr_line (start 248.239875 39.757625) (end 264.908625 39.757625) (layer Edge.Cuts) (width 0.05))
-  (gr_line (start 243.477375 52.8545) (end 38.689875 52.8545) (layer Edge.Cuts) (width 0.05))
-  (gr_line (start 245.858625 42.138875) (end 245.858625 50.47325) (layer Edge.Cuts) (width 0.05))
-  (gr_arc (start 243.477375 50.47325) (end 243.477375 52.8545) (angle -90) (layer Edge.Cuts) (width 0.05))
-  (gr_arc (start 254.193 48.092) (end 254.193 45.71075) (angle -90) (layer Edge.Cuts) (width 0.05))
-  (gr_arc (start 248.239875 42.138875) (end 248.239875 39.757625) (angle -90) (layer Edge.Cuts) (width 0.05))
   (gr_arc (start 38.689875 68.332625) (end 36.308625 68.332625) (angle -90) (layer Edge.Cuts) (width 0.05))
-  (gr_line (start 36.308625 31.42325) (end 36.308625 50.47325) (layer Edge.Cuts) (width 0.05))
-  (gr_arc (start 38.689875 50.47325) (end 36.308625 50.47325) (angle -90) (layer Edge.Cuts) (width 0.05))
   (gr_arc (start 36.308625 56.426375) (end 36.308625 59.99825) (angle -48.16488004) (layer Edge.Cuts) (width 0.05))
   (gr_line (start 264.908625 89.763875) (end 38.689875 89.763875) (layer Edge.Cuts) (width 0.05))
@@
   (gr_arc (start 113.69925 95.717) (end 110.127375 95.717) (angle -180) (layer Edge.Cuts) (width 0.05))
   (gr_line (start 117.271125 95.717) (end 186.327375 95.717) (layer Edge.Cuts) (width 0.05))
-  (gr_arc (start 36.308625 27.851375) (end 36.308625 31.42325) (angle -90) (layer Edge.Cuts) (width 0.05))
-  (gr_arc (start 267.289875 27.851375) (end 263.718 27.851375) (angle -90) (layer Edge.Cuts) (width 0.05))
   (gr_arc (start 36.308625 154.057625) (end 39.8805 154.057625) (angle -90) (layer Edge.Cuts) (width 0.05))
   (gr_arc (start 267.289875 154.057625) (end 267.289875 150.48575) (angle -90) (layer Edge.Cuts) (width 0.05))
