File: rev1/acrylic/framework-acrylic-grid.kicad_pcb (KiCad board)
At the start: 2 copper layers, 238.1 x 104.8 mm, 0 parts

Commit message: Dimension acrylic
Other:
- outline, holes or cut-outs redrawn
