File: rev1/acrylic/framework-acrylic-shield.kicad_pcb (KiCad board)
At the start: 2 copper layers, 238.1 x 28.6 mm, 0 parts

Commit message: Dimension acrylic
Changed lines of the file:
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@@
   (general
     (thickness 1.6)
-    (drawings 27)
+    (drawings 29)
     (tracks 0)
     (zones 0)
@@
     (solder_mask_min_width 0.25)
     (aux_axis_origin 0 0)
-    (grid_origin 151.79925 56.426375)
+    (grid_origin 151.79925 107.623465)
     (visible_elements 7FFFF77F)
     (pcbplotparams
@@
     (diff_pair_gap 0.25)
   )
-  (gr_line (start 144.65547 52.854485) (end 158.94303 52.854485) (layer Edge.Cuts) (width 0.05))
-  (gr_line (start 32.73625 48.091965) (end 32.73675 29.042) (layer Edge.Cuts) (width 0.05))
-  (gr_line (start 43.45192 52.854485) (end 37.49877 52.854485) (layer Edge.Cuts) (width 0.05))
-  (gr_line (start 266.09973 52.854485) (end 233.95272 52.854485) (layer Edge.Cuts) (width 0.05))
-  (gr_line (start 270.86225 48.091965) (end 270.86175 29.042) (layer Edge.Cuts) (width 0.05))
-  (gr_arc (start 266.09973 48.091965) (end 266.09973 52.854485) (angle -90) (layer Edge.Cuts) (width 0.05))
-  (gr_arc (start 37.49877 48.091965) (end 32.73625 48.091965) (angle -90) (layer Edge.Cuts) (width 0.05))
-  (gr_line (start 203.79925 24.2795) (end 249.79925 24.2795) (layer Edge.Cuts) (width 0.05))
-  (gr_line (start 153.79925 24.2795) (end 199.79925 24.2795) (layer Edge.Cuts) (width 0.05))
-  (gr_line (start 37.49925 24.2795) (end 49.79925 24.2795) (layer Edge.Cuts) (width 0.05))
-  (gr_line (start 253.79925 24.2795) (end 266.09925 24.2795) (layer Edge.Cuts) (width 0.05))
-  (gr_line (start 103.79925 24.2795) (end 149.79925 24.2795) (layer Edge.Cuts) (width 0.05))
-  (gr_line (start 53.79925 24.2795) (end 99.79925 24.2795) (layer Edge.Cuts) (width 0.05))
-  (gr_arc (start 37.49925 29.042) (end 37.49925 24.2795) (angle -90) (layer Edge.Cuts) (width 0.05))
-  (gr_arc (start 266.09925 29.042) (end 270.86175 29.042) (angle -90) (layer Edge.Cuts) (width 0.05))
-  (gr_circle (center 36.308625 27.851375) (end 37.408625 27.851375) (layer Edge.Cuts) (width 0.05))
-  (gr_line (start 43.45192 52.854485) (end 144.65547 52.854485) (layer Edge.Cuts) (width 0.05))
-  (gr_circle (center 267.29036 49.282595) (end 268.39036 49.282595) (layer Edge.Cuts) (width 0.05))
-  (gr_line (start 233.95272 52.854485) (end 158.94303 52.854485) (layer Edge.Cuts) (width 0.05))
-  (gr_circle (center 36.30814 49.282595) (end 37.40814 49.282595) (layer Edge.Cuts) (width 0.05))
-  (gr_circle (center 151.79925 48.091965) (end 152.89925 48.091965) (layer Edge.Cuts) (width 0.05))
-  (gr_circle (center 267.289875 27.851375) (end 268.389875 27.851375) (layer Edge.Cuts) (width 0.05))
-  (gr_arc (start 266.09925 29.042) (end 270.86175 29.042) (angle -90) (layer Edge.Cuts) (width 0.05))
-  (gr_line (start 37.49925 24.2795) (end 49.79925 24.2795) (layer Edge.Cuts) (width 0.05))
-  (gr_line (start 253.79925 24.2795) (end 266.09925 24.2795) (layer Edge.Cuts) (width 0.05))
-  (gr_arc (start 37.49925 29.042) (end 37.49925 24.2795) (angle -90) (layer Edge.Cuts) (width 0.05))
-  (gr_line (start 49.79925 24.2795) (end 253.79925 24.2795) (layer Edge.Cuts) (width 0.05))
+  (dimension 238.126 (width 0.12) (layer F.SilkS)
+    (gr_text "238.126 mm" (at 151.79925 117.227875) (layer F.SilkS)
+      (effects (font (size 1 1) (thickness 0.15)))
+    )
+    (feature1 (pts (xy 270.86225 107.623465) (xy 270.86225 116.544296)))
+    (feature2 (pts (xy 32.73625 107.623465) (xy 32.73625 116.544296)))
+    (crossbar (pts (xy 32.73625 115.957875) (xy 270.86225 115.957875)))
+    (arrow1a (pts (xy 270.86225 115.957875) (xy 269.735746 116.544296)))
+    (arrow1b (pts (xy 270.86225 115.957875) (xy 269.735746 115.371454)))
+    (arrow2a (pts (xy 32.73625 115.957875) (xy 33.862754 116.544296)))
+    (arrow2b (pts (xy 32.73625 115.957875) (xy 33.862754 115.371454)))
+  )
+  (dimension 28.574985 (width 0.12) (layer F.SilkS)
+    (gr_text "28.575 mm" (at 27.894601 98.098331 89.99903755) (layer F.SilkS)
+      (effects (font (size 1 1) (thickness 0.15)))
+    )
+    (feature1 (pts (xy 37.49877 112.385985) (xy 28.57794 112.385835)))
+    (feature2 (pts (xy 37.49925 83.811) (xy 28.57842 83.81085)))
+    (crossbar (pts (xy 29.164841 83.81086) (xy 29.164361 112.385845)))
+    (arrow1a (pts (xy 29.164361 112.385845) (xy 28.577959 111.259331)))
+    (arrow1b (pts (xy 29.164361 112.385845) (xy 29.750801 111.259351)))
+    (arrow2a (pts (xy 29.164841 83.81086) (xy 28.578401 84.937354)))
+    (arrow2b (pts (xy 29.164841 83.81086) (xy 29.751243 84.937374)))
+  )
+  (gr_line (start 144.65547 112.385985) (end 158.94303 112.385985) (layer Edge.Cuts) (width 0.05))
+  (gr_line (start 32.73625 107.623465) (end 32.73675 88.5735) (layer Edge.Cuts) (width 0.05))
+  (gr_line (start 43.45192 112.385985) (end 37.49877 112.385985) (layer Edge.Cuts) (width 0.05))
+  (gr_line (start 266.09973 112.385985) (end 233.95272 112.385985) (layer Edge.Cuts) (width 0.05))
+  (gr_line (start 270.86225 107.623465) (end 270.86175 88.5735) (layer Edge.Cuts) (width 0.05))
+  (gr_arc (start 266.09973 107.623465) (end 266.09973 112.385985) (angle -90) (layer Edge.Cuts) (width 0.05))
+  (gr_arc (start 37.49877 107.623465) (end 32.73625 107.623465) (angle -90) (layer Edge.Cuts) (width 0.05))
+  (gr_line (start 203.79925 83.811) (end 249.79925 83.811) (layer Edge.Cuts) (width 0.05))
+  (gr_line (start 153.79925 83.811) (end 199.79925 83.811) (layer Edge.Cuts) (width 0.05))
+  (gr_line (start 37.49925 83.811) (end 49.79925 83.811) (layer Edge.Cuts) (width 0.05))
+  (gr_line (start 253.79925 83.811) (end 266.09925 83.811) (layer Edge.Cuts) (width 0.05))
+  (gr_line (start 103.79925 83.811) (end 149.79925 83.811) (layer Edge.Cuts) (width 0.05))
+  (gr_line (start 53.79925 83.811) (end 99.79925 83.811) (layer Edge.Cuts) (width 0.05))
+  (gr_arc (start 37.49925 88.5735) (end 37.49925 83.811) (angle -90) (layer Edge.Cuts) (width 0.05))
+  (gr_arc (start 266.09925 88.5735) (end 270.86175 88.5735) (angle -90) (layer Edge.Cuts) (width 0.05))
+  (gr_circle (center 36.308625 87.382875) (end 37.408625 87.382875) (layer Edge.Cuts) (width 0.05))
+  (gr_line (start 43.45192 112.385985) (end 144.65547 112.385985) (layer Edge.Cuts) (width 0.05))
+  (gr_circle (center 267.29036 108.814095) (end 268.39036 108.814095) (layer Edge.Cuts) (width 0.05))
+  (gr_line (start 233.95272 112.385985) (end 158.94303 112.385985) (layer Edge.Cuts) (width 0.05))
+  (gr_circle (center 36.30814 108.814095) (end 37.40814 108.814095) (layer Edge.Cuts) (width 0.05))
+  (gr_circle (center 151.79925 107.623465) (end 152.89925 107.623465) (layer Edge.Cuts) (width 0.05))
+  (gr_circle (center 267.289875 87.382875) (end 268.389875 87.382875) (layer Edge.Cuts) (width 0.05))
+  (gr_arc (start 266.09925 88.5735) (end 270.86175 88.5735) (angle -90) (layer Edge.Cuts) (width 0.05))
+  (gr_line (start 37.49925 83.811) (end 49.79925 83.811) (layer Edge.Cuts) (width 0.05))
+  (gr_line (start 253.79925 83.811) (end 266.09925 83.811) (layer Edge.Cuts) (width 0.05))
+  (gr_arc (start 37.49925 88.5735) (end 37.49925 83.811) (angle -90) (layer Edge.Cuts) (width 0.05))
+  (gr_line (start 49.79925 83.811) (end 253.79925 83.811) (layer Edge.Cuts) (width 0.05))
 )
